File: Hardware/schematic.sch (EAGLE design)
At the start: 105 parts, among them IC1 BQ25180YBGR, IC2 DRV2605YZFR, IC3 BMA423, IC9 RT6160AWSC, J1 503480-2400, J2 TC2030-IDC_TC2030-IDC, J4 KH-TYPE-C-16P, Q1 SI1308EDL-T1-GE3, Q2 3.1A/30V/105mΩ, U1 NRF52840_QF, U3 MAX17048G+T10, X1 32MHz, X2 32.768kHz

Commit message: Schematic and 2D PCB updated to final version
Parts:
- removed Q2: 3.1A/30V/105mΩ, InkTime_v5:ESP32_C6_LIBRARY_4_ESP32_WROVER_SPARKFUN-DISCRETESEMI_MOSFET_PCH-DMG2307L
- added Q3: SI1308EDL-T1-GE3, InkTime_v5:ESP32_C6_LIBRARY_6_SI1308EDL-T1-GE3
- Q1: value SI1308EDL-T1-GE3 -> 3.1A/30V/105mΩ; device InkTime_v5:ESP32_C6_LIBRARY_6_SI1308EDL-T1-GE3 -> InkTime_v5:ESP32_C6_LIBRARY_4_ESP32_WROVER_SPARKFUN-DISCRETESEMI_MOSFET_PCH-DMG2307L
- U$1: value NRF52840_QF -> NORDIC_NRF_4_NRF52840_QF
- renumbered D1 to D3, TP_3.3V to 3.3V, TP_3V3 to 3V3, TP_BAT_GND to BAT_GND, TP_GND to GND, TP_ON to ON, TP_OP to OP, TP_RESET to RESET, TP_SCL to SCL, TP_SDA to SDA, TP_SWDCLK to SWDCLK, TP_SWDIO to SWDIO, TP_SWO to SWO, TP_VBAT to VBAT, TP_VREG to VREG, U1 to U$1
Connections:
- net N$9 renamed 3.3V
- removed net 3V3/1.7D: C34.1, IC2.VDD, Q2.S, R5.2, R7.2, R8.2, R_PWR_EPD.2
- removed net 3V3/2.4A: 3.3V.TP, 3V3.TP, C12.1, C14.1, C19.1, C6.1, C7.1, C8.1, IC3.CSB, IC3.VDD, IC3.VDDIO, J2.1, R17.1, R18.1, U$1.VDD@A22, U$1.VDD@AD14, U$1.VDD@AD23, U$1.VDD@B1, U$1.VDD@W1, U$1.VDDH@Y2
- removed net ALERT/1.6C: U3.!ALERT
- removed net ALERT/2.5C: U$1.P0.10/NFC2@J24
- removed net D+/1.5D: D3.I/O2_2
- removed net D+/2.7D: U$1.D+@AD6
- removed net D-/1.5D: D3.I/O1_2
- removed net D-/2.7D: U$1.D-@AD4
- removed net EPD_BUSY/1.5D: J1.9
- removed net EPD_BUSY/2.2D: U$1.P0.17@AD12
- removed net EPD_CS/1.4C: J1.12
- removed net EPD_CS/2.2D: U$1.P0.05/AIN3@K2
- removed net EPD_DC/1.5D: J1.11
- removed net EPD_DC/2.2D: U$1.P0.15@AD10
- removed net EPD_RST/1.5D: J1.10
- removed net EPD_RST/2.2D: U$1.P0.16@AC11
- removed net HAPTIC_EN/1.4C: IC2.EN
- removed net HAPTIC_EN/2.6A: U$1.P0.12@U1
- removed net MOSI/1.5B: J1.14
- removed net MOSI/2.2D: U$1.P0.03/AIN1@B13
- removed net P0.13/1.5D: C30.1, R5.1, SW_UP.2
- removed net P0.13/2.6C: U$1.P0.13@AD8
- removed net P0.14/1.5D: C31.1, R8.1, SW_ENT.2
- removed net P0.14/2.7C: U$1.P0.14@AC9
- removed net P1.01/1.6C: Q2.G, R_PWR_EPD.1
- removed net P1.01/2.4B: U$1.P1.01@Y23
- removed net P1.02/1.6C: C29.1, R7.1, SW_DN.2
- removed net P1.02/2.8C: U$1.P1.02@W24
- removed net SCK/1.5B: J1.13
- removed net SCK/2.2D: U$1.P0.02/AIN0@A12
- removed net SCL/1.4C: IC2.SCL, U3.SCL
- removed net SCL/2.4C: IC1.SCL, IC3.SCX, R17.2, R4.1, SCL.TP, U$1.P0.07@M2
- removed net SDA/1.4C: IC2.SDA, U3.SDA
- removed net SDA/2.4C: IC1.SDA, IC3.SDX, R1.1, R18.2, SDA.TP, U$1.P0.06@L1
- removed net VBAT/1.2A: C27.1, U3.CELL, U3.VDD, VBAT.TP
- removed net VBAT/2.5C: C37.1, IC1.BAT
- removed net VBUS/1.5D: C42.1, C43.1, D3.VBUS, J4.VBUS
- removed net VBUS/2.6D: C21.1, C38.1, IC1.IN, U$1.VBUS@AD2
- new net 3V3: 3.3V.TP, 3V3.TP, C12.1, C14.1, C19.1, C34.1, C6.1, C7.1, C8.1, IC2.VDD, IC3.CSB, IC3.VDD, IC3.VDDIO, J2.1, Q1.S, R17.1, R18.1, R5.2, R7.2, R8.2, R_PWR_EPD.2, U$1.VDD@A22, U$1.VDD@AD14, U$1.VDD@AD23, U$1.VDD@B1, U$1.VDD@W1, U$1.VDDH@Y2
- new net ALERT: U$1.P0.10/NFC2@J24, U3.!ALERT
- new net D+: D3.I/O2_2, U$1.D+@AD6
- new net D-: D3.I/O1_2, U$1.D-@AD4
- new net EPD_BUSY: J1.9, U$1.P0.17@AD12
- new net EPD_CS: J1.12, U$1.P0.05/AIN3@K2
- new net EPD_DC: J1.11, U$1.P0.15@AD10
- new net EPD_RST: J1.10, U$1.P0.16@AC11
- new net HAPTIC_EN: IC2.EN, U$1.P0.12@U1
- new net MOSI: J1.14, U$1.P0.03/AIN1@B13
- new net P0.13: C30.1, R5.1, SW_UP.2, U$1.P0.13@AD8
- new net P0.14: C31.1, R8.1, SW_ENT.2, U$1.P0.14@AC9
- new net P1.01: Q1.G, R_PWR_EPD.1, U$1.P1.01@Y23
- new net P1.02: C29.1, R7.1, SW_DN.2, U$1.P1.02@W24
- new net SCK: J1.13, U$1.P0.02/AIN0@A12
- new net SCL: IC1.SCL, IC2.SCL, IC3.SCX, R17.2, R4.1, SCL.TP, U$1.P0.07@M2, U3.SCL
- new net SDA: IC1.SDA, IC2.SDA, IC3.SDX, R1.1, R18.2, SDA.TP, U$1.P0.06@L1, U3.SDA
- new net VBAT: C27.1, C37.1, IC1.BAT, U3.CELL, U3.VDD, VBAT.TP
- new net VBUS: C21.1, C38.1, C42.1, C43.1, D3.VBUS, IC1.IN, J4.VBUS, U$1.VBUS@AD2
- net EPD_3V3: now also Q1.D; no longer Q2.D
- net GDR: now also Q3.G; no longer Q1.G
- net GND: now also C23.1; no longer C23.2
- net N$17: now also Q3.D; no longer Q1.D
- net RESE: now also Q3.S; no longer Q1.S
- net VREG: now also C23.2; no longer C23.1
Other:
- moved on the sheet: C23
